Commit message: Migrating local changes

File: robosuite/models/assets/bullet_data/panda_description/urdf/panda_arm.xacro (robot description, xacro)
@@ -45,5 +45,5 @@
     <joint name="${arm_id}_joint1" type="revolute">
       <safety_controller k_position="100.0" k_velocity="40.0" soft_lower_limit="-2.8973" soft_upper_limit="2.8973"/>
-      <origin rpy="0 0 0" xyz="0 0 0.333"/>
+      <origin rpy="0 0 0" xyz="0 -0.1 0"/>
       <parent link="${arm_id}_link0"/>
       <child link="${arm_id}_link1"/>

File: robosuite/models/assets/bullet_data/panda_description/urdf/panda_arm_hand.urdf (robot description, URDF)
Before this commit: robot panda, 12 links, 11 joints
Joints:
- joint panda_joint1: origin xyz=0 0 0.333 rpy=0 0 0 -> xyz=0 -0.1 0 rpy=0 0 0
